Commit message: Fix orientation and cleanup

File: src/onrobot_rg6_visualization/urdf/onrobot_rg6.xacro (robot description, xacro)
@@ -13,5 +13,5 @@
           <mesh filename="package://onrobot_rg6_visualization/meshes/visual/base_link.stl" />
         </geometry>
-        <material name="">
+        <material name="rg6_silver">
           <color rgba="0.8 0.8 0.8 1" />
         </material>

File: src/onrobot_rg6_visualization/urdf/onrobot_rg6_model_macro.xacro (robot description, xacro)
@@ -1,5 +1,7 @@
 <?xml version="1.0"?>
 <robot xmlns:xacro="http://ros.org/wiki/xacro">
-  <xacro:include filename="$(find onrobot_rg6_visualization)/urdf/onrobot_rg6_transmission.xacro" />
+  <!-- transmission/mimic bewusst entfernt: der rg6_joint_state_broadcaster treibt
+       alle 6 Gelenke explizit. Manche URDF-Parser (z.B. Foxglove) stolpern ueber
+       <mimic>/<transmission>/leere Material-Namen -> Meshes landen im Ursprung. -->
   <xacro:macro name="outer_knuckle" params="prefix fingerprefix">
     <link name="${prefix}${fingerprefix}_outer_knuckle">
@@ -14,5 +16,5 @@
           <mesh filename="package://onrobot_rg6_visualization/meshes/visual/outer_knuckle.stl" />
         </geometry>
-        <material name="">
+        <material name="rg6_silver">
           <color rgba="0.8 0.8 0.8 1" />
         </material>
@@ -38,5 +40,5 @@
           <mesh filename="package://onrobot_rg6_visualization/meshes/visual/inner_knuckle.stl" />
         </geometry>
-        <material name="">
+        <material name="rg6_silver">
           <color rgba="0.8 0.8 0.8 1" />
         </material>
@@ -62,5 +64,5 @@
           <mesh filename="package://onrobot_rg6_visualization/meshes/visual/inner_finger.stl" />
         </geometry>
-        <material name="">
+        <material name="rg6_black">
           <color rgba="0.1 0.1 0.1 1" />
         </material>
@@ -81,5 +83,4 @@
       <axis xyz="1 0 0" />
       <limit lower="-0.628319" upper="0.628319" velocity="2.0" effort="1000" />
-      <mimic joint="${prefix}finger_joint" multiplier="-1" offset="0" />
     </joint>
   </xacro:macro>
@@ -91,5 +92,4 @@
       <axis xyz="1 0 0" />
       <limit lower="-0.872665" upper="0.872665" velocity="2.0" effort="1000" />
-      <mimic joint="${prefix}finger_joint" multiplier="1" offset="0" />
     </joint>
   </xacro:macro>
@@ -112,5 +112,4 @@
       <axis xyz="1 0 0" />
       <limit lower="-0.628319" upper="0.628319" velocity="2.0" effort="1000" />
-    <mimic joint="${prefix}finger_joint" multiplier="-1" offset="0" />
     </joint>
     <xacro:finger_joints prefix="${prefix}" fingerprefix="right" reflect="-1.0"/>
@@ -122,5 +121,4 @@
     <xacro:finger_joint prefix="${prefix}"/>
     <xacro:right_outer_knuckle_joint prefix="${prefix}"/>
-    <xacro:onrobot_rg6_transmission prefix="${prefix}"/>
   </xacro:macro>
 </robot>

File: src/rg6_description/urdf/clearpath_extras.urdf.xacro (robot description, xacro)
@@ -47,5 +47,5 @@
     <parent link="arm_0_tool0"/>
     <child link="rg6_onrobot_rg6_base_link"/>
-    <origin xyz="0 0 0" rpy="-1.5708 0 0"/>
+    <origin xyz="0 0 0" rpy="0 0 0"/>
   </joint>
   <!-- Greifer-TCP (mittig zwischen den Fingerspitzen, grob). -->

Commit message: Delete self colliding elements

File: src/onrobot_rg6_visualization/urdf/onrobot_rg6.xacro (robot description, xacro)
@@ -17,10 +17,6 @@
         </material>
       </visual>
-      <collision>
-        <origin xyz="0 0 0" rpy="0 0 0" />
-        <geometry>
-          <mesh filename="package://onrobot_rg6_visualization/meshes/collision/base_link.stl" />
-        </geometry>
-      </collision>
+      <!-- collision weggelassen: Greifer ist Anzeige-only; mit collision kollidiert
+           die Basis am Flansch/Handgelenk -> MoveIt-Startzustand "in Kollision". -->
     </link>
   </xacro:macro>

File: src/onrobot_rg6_visualization/urdf/onrobot_rg6_model_macro.xacro (robot description, xacro)
@@ -20,10 +20,6 @@
         </material>
       </visual>
-      <collision>
-        <origin xyz="0 0 0" rpy="0 0 0" />
-        <geometry>
-          <mesh filename="package://onrobot_rg6_visualization/meshes/collision/outer_knuckle.stl" />
-        </geometry>
-      </collision>
+      <!-- collision bewusst weggelassen: 4-Gelenk-Schleife im URDF-Baum -> sonst
+           Selbstkollision -> MoveIt-Planung schlaegt fehl. Greifer ist Anzeige-only. -->
     </link>
   </xacro:macro>
@@ -44,10 +40,5 @@
         </material>
       </visual>
-      <collision>
-        <origin xyz="0 0 0" rpy="0 0 0" />
-        <geometry>
-          <mesh filename="package://onrobot_rg6_visualization/meshes/collision/inner_knuckle.stl" />
-        </geometry>
-      </collision>
+      <!-- collision weggelassen (siehe outer_knuckle). -->
     </link>
   </xacro:macro>
@@ -68,10 +59,5 @@
         </material>
       </visual>
-      <collision>
-        <origin xyz="0 0 0" rpy="0 0 0" />
-        <geometry>
-          <mesh filename="package://onrobot_rg6_visualization/meshes/collision/inner_finger.stl" />
-        </geometry>
-      </collision>
+      <!-- collision weggelassen (siehe outer_knuckle). -->
     </link>
   </xacro:macro>

Commit message: Add collisions for moveit

File: src/onrobot_rg6_visualization/urdf/onrobot_rg6.xacro (robot description, xacro)
@@ -17,6 +17,17 @@
         </material>
       </visual>
-      <!-- collision weggelassen: Greifer ist Anzeige-only; mit collision kollidiert
-           die Basis am Flansch/Handgelenk -> MoveIt-Startzustand "in Kollision". -->
+      <!-- EINE grobe Huell-Box fuer den GANZEN Greifer (Basis+Finger), statt
+           filigraner Einzel-Meshes. Ein einziger Kollisionskoerper -> keine
+           Selbstkollision (war die MoveIt-Planungsblockade), aber Greifer wird
+           gegen Arm/Umgebung geprueft. Box liegt +z (vor dem Flansch), reicht
+           NICHT in arm_0_wrist_3_link zurueck -> kein Handgelenk-Falschtreffer.
+           Masse aus Greifer-Huellmass (offen): x +-0.05, y +-0.09, z 0.02..0.27.
+           Bei Bedarf in RViz (Collision Enabled) nachziehen. -->
+      <collision>
+        <origin xyz="0 0 0.145" rpy="0 0 0"/>
+        <geometry>
+          <box size="0.11 0.19 0.25"/>
+        </geometry>
+      </collision>
     </link>
   </xacro:macro>

File: src/rg6_description/urdf/clearpath_extras.urdf.xacro (robot description, xacro)
@@ -58,15 +58,19 @@
   <link name="husky_top_assembly">
     <visual>
-      <origin xyz="0 0 0" rpy="0 0 0"/>
+      <!-- Visual-Origin "nullt" das Mesh: rpy dreht es aufrecht, xyz schiebt den
+           Fuss-Mittelpunkt auf den Link-Ursprung (CAD-Versatz nach Drehung:
+           x 0.31, y 0.30, z -0.265 -> Gegenvektor hier). -->
+      <origin xyz="-0.31 -0.30 0.265" rpy="-1.5708 0 0"/>
       <geometry>
         <mesh filename="package://onrobot_rg6_visualization/meshes/husky_sensor_arch.stl"/>
-        <!-- falls nicht in Metern exportiert: scale="0.001 0.001 0.001" am mesh ergaenzen -->
       </geometry>
     </visual>
   </link>
   <joint name="husky_top_assembly_joint" type="fixed">
-    <parent link="default_mount"/>      <!-- TODO: realer Mount-Frame aus Schritt 1 -->
+    <parent link="top_plate_back_mount"/>
     <child link="husky_top_assembly"/>
-    <origin xyz="0 0 0" rpy="0 0 0"/>   <!-- TODO: Offset aus Schritt 1 -->
+    <!-- Origin 0 0 0 = Fuss-Mittelpunkt sitzt exakt auf top_plate_back_mount.
+         Hier intuitiv nachschieben (z hoch, x vor/zurueck, y links/rechts). -->
+    <origin xyz="0 0 0" rpy="0 0 0"/>
   </joint>
 </robot>
