Commit message: Fix RG6 orientation

File: src/rg6_description/urdf/clearpath_extras.urdf.xacro (robot description, xacro)
@@ -37,8 +37,10 @@
   </joint>
   <!-- ===================== RG6-Greifer an arm_0_tool0 =================== -->
+  <!-- rpy korrigiert die Verkippung am Tool-Flansch: Roll -90deg um X
+       (empirisch bestaetigt fuer arm_0_tool0 auf diesem Roboter). -->
   <joint name="rg6_tool0_to_base" type="fixed">
     <parent link="arm_0_tool0"/>
     <child link="rg6_base_link"/>
-    <origin xyz="0 0 0" rpy="0 0 0"/>
+    <origin xyz="0 0 0" rpy="-1.5708 0 0"/>
   </joint>
   <link name="rg6_base_link">

Commit message: Add RG6 animation

File: src/rg6_description/urdf/clearpath_extras.urdf.xacro (robot description, xacro)
@@ -108,32 +108,52 @@
     </visual>
   </link>
-  <!-- Gelenke: hier FIXED in Nominalpose (Offsets = die der Originalgelenke). -->
+  <!-- Gelenke: g_main + hand_tcp fixed; Finger revolute+mimic fuer Auf/Zu-Animation.
+       TREIBER = 'rg6-l_out_joint' (Bindestrich!) -> exakt der Name, den der
+       rg6_joint_state_broadcaster publiziert. Alle anderen Finger folgen per <mimic>,
+       brauchen also KEINE eigene joint_states-Quelle. axis/limit/mimic wie im Original. -->
   <joint name="rg6_g_main_joint" type="fixed">
     <origin xyz="-0.031849 1e-06 0.04953" rpy="0 0 0"/>
     <parent link="rg6_base_link"/><child link="rg6_g_main"/>
   </joint>
-  <joint name="rg6_l_out_joint" type="fixed">
+  <joint name="rg6-l_out_joint" type="revolute">
     <origin xyz="0.0557 0.0128 0.085" rpy="0 0 0"/>
     <parent link="rg6_g_main"/><child link="rg6_l_out"/>
+    <axis xyz="0 1 0"/>
+    <limit upper="0.610865" lower="-0.75" effort="100" velocity="100"/>
   </joint>
-  <joint name="rg6_r_out_joint" type="fixed">
+  <joint name="rg6_r_out_joint" type="revolute">
     <origin xyz="0.0081 0.0128 0.085" rpy="0 0 0"/>
     <parent link="rg6_g_main"/><child link="rg6_r_out"/>
+    <axis xyz="0 1 0"/>
+    <limit upper="0.523599" lower="-0.610865" effort="100" velocity="100"/>
+    <mimic joint="rg6-l_out_joint" multiplier="-1"/>
   </joint>
-  <joint name="rg6_l_tip_joint" type="fixed">
+  <joint name="rg6_l_tip_joint" type="revolute">
     <origin xyz="0.047384 -0.0253 0.06442" rpy="0 0 0"/>
     <parent link="rg6_l_out"/><child link="rg6_l_tip"/>
+    <axis xyz="0 -1 0"/>
+    <limit upper="0.610865" lower="-0.523599" effort="100" velocity="100"/>
+    <mimic joint="rg6-l_out_joint" multiplier="1"/>
   </joint>
-  <joint name="rg6_r_tip_joint" type="fixed">
+  <joint name="rg6_r_tip_joint" type="revolute">
     <origin xyz="-0.047384 -0.0253 0.064494" rpy="0 0 0"/>
     <parent link="rg6_r_out"/><child link="rg6_r_tip"/>
+    <axis xyz="0 -1 0"/>
+    <limit upper="0.523599" lower="-0.610865" effort="100" velocity="100"/>
+    <mimic joint="rg6-l_out_joint" multiplier="-1"/>
   </joint>
-  <joint name="rg6_l_passive_joint" type="fixed">
+  <joint name="rg6_l_passive_joint" type="revolute">
     <origin xyz="0.0424 0.0001 0.1081" rpy="0 0 0"/>
     <parent link="rg6_g_main"/><child link="rg6_l_inner"/>
+    <axis xyz="0 -1 0"/>
+    <limit upper="0.523599" lower="-0.610865" effort="100" velocity="100"/>
+    <mimic joint="rg6-l_out_joint" multiplier="-1"/>
   </joint>
-  <joint name="rg6_r_passive_joint" type="fixed">
+  <joint name="rg6_r_passive_joint" type="revolute">
     <origin xyz="0.0214 0.0001 0.1081" rpy="0 0 0"/>
     <parent link="rg6_g_main"/><child link="rg6_r_inner"/>
+    <axis xyz="0 1 0"/>
+    <limit upper="0.523599" lower="-0.610865" effort="100" velocity="100"/>
+    <mimic joint="rg6-l_out_joint" multiplier="-1"/>
   </joint>
   <!-- Greifer-TCP -->
@@ -144,8 +164,9 @@
   </joint>
   <!--
-    AUF/ZU-ANIMATION (optional): die 'fixed'-Greifer-Gelenke wieder auf 'revolute'
-    mit axis/limit/mimic wie im Original setzen (rg6_l_out_joint als Treiber,
-    die anderen mit <mimic joint="rg6_l_out_joint" .../>). Dann braucht es aber
-    eine joint_states-Quelle fuer rg6_l_out_joint, sonst meckert robot_state_publisher.
+    AUF/ZU-ANIMATION: aktiv. Treiber 'rg6-l_out_joint' wird vom
+    rg6_joint_state_broadcaster aus tool_data.analog_input2 gespeist. Damit der
+    Greifer animiert, muss dessen joint_states auf dem Topic landen, das der
+    Greifer-rendernde robot_state_publisher konsumiert (siehe rg6_bringup.launch.py
+    Argument 'js_topic').
   -->
 </robot>

Commit message: Fix RG6 model issue

File: src/rg6_description/urdf/clearpath_extras.urdf.xacro (robot description, xacro)
@@ -6,15 +6,23 @@
         extras:
           urdf:
-            path: /home/robot/colcon_ws/.../clearpath_extras.urdf.xacro
-  (Pfad an deinen Ablageort anpassen; Datei muss vom Generator lesbar sein.)
+            path: /home/robot/onrobot-rg6/.../clearpath_extras.urdf.xacro
   Haengt NUR neue Links/Joints an bereits vom Generator erzeugte Frames an:
     - arm_0_tool0   = UR5 Tool-Frame (ROS-Industrial all-zeros)  -> RG6-Greifer
-    - <MARKER_PARENT> = Frame, auf dem der ArUco-Marker physisch sitzt
+    - default_mount = Frame, auf dem der ArUco-Marker sitzt (TODO anpassen)
   WICHTIG:
-    * Alle Greifer-Links sind mit 'rg6_' praefixiert -> KEINE Kollision mit
-      dem Husky 'base_link'.
+    * Alle Greifer-Links sind mit 'rg6_' praefixiert -> KEINE Kollision mit base_link.
     * rg6_description muss in einem in robot.yaml eingetragenen Workspace liegen.
-    * Greifer-Gelenke hier als 'fixed' (Nominalpose) -> rendert zuverlaessig ohne
-      eigene joint_states. Fuer echte Auf/Zu-Animation siehe Hinweis unten.
+  ANIMATION (Auf/Zu):
+    Die RG6-Meshes sind im SolidWorks-Export ALLE im Basis-Frame authored (jedes
+    Mesh sitzt korrekt, wenn es bei xyz=0 an rg6_base_link haengt). Die reale
+    Kinematik ist ein 4-Gelenk-Parallelogramm pro Finger; das laesst sich im
+    URDF-Baum nur ungenau per mimic abbilden und ZERFAELLT bei Bewegung.
+    Daher hier vereinfacht: jeder Finger = EIN starrer Link (out+tip+inner), der um
+    sein Aussengelenk schwenkt. Treibergelenk 'rg6-l_out_joint' wird vom
+    rg6_joint_state_broadcaster aus tool_data.analog_input2 gespeist; der rechte
+    Finger folgt per <mimic multiplier="-1"> -> symmetrisches Auf/Zu, nichts zerfaellt.
+    Pivot/Visual-Offsets sind die globalen Aussengelenk-Positionen:
+        links  = base->g_main + g_main->l_out = (0.023851, 0.012801, 0.13453)
+        rechts = base->g_main + g_main->r_out = (-0.023749, 0.012801, 0.13453)
 -->
 <robot xmlns:xacro="http://ros.org/wiki/xacro">
@@ -23,6 +31,5 @@
   <material name="white"><color rgba="0.9137 0.9137 0.9137 1.0"/></material>
   <!-- =========================== ArUco-Marker =========================== -->
-  <!-- TODO: MARKER_PARENT + Offset an die reale Position anpassen.
-       Im Altmodell war der Marker an 'robot_mount' mit xyz 0.048 -0.134 0. -->
+  <!-- TODO: MARKER_PARENT + Offset an die reale Position anpassen. -->
   <link name="aruco_marker">
     <visual>
@@ -37,6 +44,5 @@
   </joint>
   <!-- ===================== RG6-Greifer an arm_0_tool0 =================== -->
-  <!-- rpy korrigiert die Verkippung am Tool-Flansch: Roll -90deg um X
-       (empirisch bestaetigt fuer arm_0_tool0 auf diesem Roboter). -->
+  <!-- rpy: Roll -90deg um X (empirisch bestaetigt fuer arm_0_tool0). -->
   <joint name="rg6_tool0_to_base" type="fixed">
     <parent link="arm_0_tool0"/>
@@ -44,4 +50,5 @@
     <origin xyz="0 0 0" rpy="-1.5708 0 0"/>
   </joint>
+  <!-- ===== statische Teile ===== -->
   <link name="rg6_base_link">
     <visual>
@@ -66,5 +73,6 @@
     </collision>
   </link>
-  <link name="rg6_l_out">
+  <!-- ===== linker Finger als EIN starrer Link (out + tip + inner) ===== -->
+  <link name="rg6_left_finger">
     <visual>
       <origin xyz="-0.023851 -0.012801 -0.13453" rpy="0 0 0"/>
@@ -72,6 +80,25 @@
       <material name="silver"/>
     </visual>
+    <visual>
+      <origin xyz="-0.023851 -0.012801 -0.13453" rpy="0 0 0"/>
+      <geometry><mesh filename="package://rg6_description/meshes/l_inner.stl" scale="0.001 0.001 0.001"/></geometry>
+      <material name="silver"/>
+    </visual>
+    <visual>
+      <origin xyz="-0.023851 -0.012801 -0.13453" rpy="0 0 0"/>
+      <geometry><mesh filename="package://rg6_description/meshes/l_tip.stl" scale="0.001 0.001 0.001"/></geometry>
+      <material name="black"/>
+    </visual>
+    <collision>
+      <origin xyz="-0.023851 -0.012801 -0.13453" rpy="0 0 0"/>
+      <geometry><mesh filename="package://rg6_description/meshes/l_out.stl" scale="0.001 0.001 0.001"/></geometry>
+    </collision>
+    <collision>
+      <origin xyz="-0.023851 -0.012801 -0.13453" rpy="0 0 0"/>
+      <geometry><mesh filename="package://rg6_description/meshes/l_tip.stl" scale="0.001 0.001 0.001"/></geometry>
+    </collision>
   </link>
-  <link name="rg6_r_out">
+  <!-- ===== rechter Finger als EIN starrer Link (out + tip + inner) ===== -->
+  <link name="rg6_right_finger">
     <visual>
       <origin xyz="0.023749 -0.012801 -0.13453" rpy="0 0 0"/>
@@ -79,80 +106,40 @@
       <material name="silver"/>
     </visual>
-  </link>
-  <link name="rg6_l_tip">
     <visual>
-      <origin xyz="-0.071235 0.012499 -0.19895" rpy="0 0 0"/>
-      <geometry><mesh filename="package://rg6_description/meshes/l_tip.stl" scale="0.001 0.001 0.001"/></geometry>
-      <material name="black"/>
+      <origin xyz="0.023749 -0.012801 -0.13453" rpy="0 0 0"/>
+      <geometry><mesh filename="package://rg6_description/meshes/r_inner.stl" scale="0.001 0.001 0.001"/></geometry>
+      <material name="silver"/>
     </visual>
-  </link>
-  <link name="rg6_r_tip">
     <visual>
-      <origin xyz="0.071133 0.012499 -0.199024" rpy="0 0 0"/>
+      <origin xyz="0.023749 -0.012801 -0.13453" rpy="0 0 0"/>
       <geometry><mesh filename="package://rg6_description/meshes/r_tip.stl" scale="0.001 0.001 0.001"/></geometry>
       <material name="black"/>
     </visual>
+    <collision>
+      <origin xyz="0.023749 -0.012801 -0.13453" rpy="0 0 0"/>
+      <geometry><mesh filename="package://rg6_description/meshes/r_out.stl" scale="0.001 0.001 0.001"/></geometry>
+    </collision>
+    <collision>
+      <origin xyz="0.023749 -0.012801 -0.13453" rpy="0 0 0"/>
+      <geometry><mesh filename="package://rg6_description/meshes/r_tip.stl" scale="0.001 0.001 0.001"/></geometry>
+    </collision>
   </link>
-  <link name="rg6_l_inner">
-    <visual>
-      <origin xyz="-0.010551 -0.000101 -0.15763" rpy="0 0 0"/>
-      <geometry><mesh filename="package://rg6_description/meshes/l_inner.stl" scale="0.001 0.001 0.001"/></geometry>
-      <material name="silver"/>
-    </visual>
-  </link>
-  <link name="rg6_r_inner">
-    <visual>
-      <origin xyz="0.010449 -0.000101 -0.15763" rpy="0 0 0"/>
-      <geometry><mesh filename="package://rg6_description/meshes/r_inner.stl" scale="0.001 0.001 0.001"/></geometry>
-      <material name="silver"/>
-    </visual>
-  </link>
-  <!-- Gelenke: g_main + hand_tcp fixed; Finger revolute+mimic fuer Auf/Zu-Animation.
-       TREIBER = 'rg6-l_out_joint' (Bindestrich!) -> exakt der Name, den der
-       rg6_joint_state_broadcaster publiziert. Alle anderen Finger folgen per <mimic>,
-       brauchen also KEINE eigene joint_states-Quelle. axis/limit/mimic wie im Original. -->
+  <!-- ===== Gelenke ===== -->
   <joint name="rg6_g_main_joint" type="fixed">
     <origin xyz="-0.031849 1e-06 0.04953" rpy="0 0 0"/>
     <parent link="rg6_base_link"/><child link="rg6_g_main"/>
   </joint>
+  <!-- TREIBER: vom rg6_joint_state_broadcaster gesetzt. Pivot = linkes Aussengelenk. -->
   <joint name="rg6-l_out_joint" type="revolute">
-    <origin xyz="0.0557 0.0128 0.085" rpy="0 0 0"/>
-    <parent link="rg6_g_main"/><child link="rg6_l_out"/>
+    <origin xyz="0.023851 0.012801 0.13453" rpy="0 0 0"/>
+    <parent link="rg6_base_link"/><child link="rg6_left_finger"/>
     <axis xyz="0 1 0"/>
     <limit upper="0.610865" lower="-0.75" effort="100" velocity="100"/>
   </joint>
-  <joint name="rg6_r_out_joint" type="revolute">
-    <origin xyz="0.0081 0.0128 0.085" rpy="0 0 0"/>
-    <parent link="rg6_g_main"/><child link="rg6_r_out"/>
+  <joint name="rg6_right_finger_joint" type="revolute">
+    <origin xyz="-0.023749 0.012801 0.13453" rpy="0 0 0"/>
+    <parent link="rg6_base_link"/><child link="rg6_right_finger"/>
     <axis xyz="0 1 0"/>
-    <limit upper="0.523599" lower="-0.610865" effort="100" velocity="100"/>
-    <mimic joint="rg6-l_out_joint" multiplier="-1"/>
-  </joint>
-  <joint name="rg6_l_tip_joint" type="revolute">
-    <origin xyz="0.047384 -0.0253 0.06442" rpy="0 0 0"/>
-    <parent link="rg6_l_out"/><child link="rg6_l_tip"/>
-    <axis xyz="0 -1 0"/>
-    <limit upper="0.610865" lower="-0.523599" effort="100" velocity="100"/>
-    <mimic joint="rg6-l_out_joint" multiplier="1"/>
-  </joint>
-  <joint name="rg6_r_tip_joint" type="revolute">
-    <origin xyz="-0.047384 -0.0253 0.064494" rpy="0 0 0"/>
-    <parent link="rg6_r_out"/><child link="rg6_r_tip"/>
-    <axis xyz="0 -1 0"/>
-    <limit upper="0.523599" lower="-0.610865" effort="100" velocity="100"/>
-    <mimic joint="rg6-l_out_joint" multiplier="-1"/>
-  </joint>
-  <joint name="rg6_l_passive_joint" type="revolute">
-    <origin xyz="0.0424 0.0001 0.1081" rpy="0 0 0"/>
-    <parent link="rg6_g_main"/><child link="rg6_l_inner"/>
-    <axis xyz="0 -1 0"/>
-    <limit upper="0.523599" lower="-0.610865" effort="100" velocity="100"/>
-    <mimic joint="rg6-l_out_joint" multiplier="-1"/>
-  </joint>
-  <joint name="rg6_r_passive_joint" type="revolute">
-    <origin xyz="0.0214 0.0001 0.1081" rpy="0 0 0"/>
-    <parent link="rg6_g_main"/><child link="rg6_r_inner"/>
-    <axis xyz="0 1 0"/>
-    <limit upper="0.523599" lower="-0.610865" effort="100" velocity="100"/>
+    <limit upper="0.610865" lower="-0.75" effort="100" velocity="100"/>
     <mimic joint="rg6-l_out_joint" multiplier="-1"/>
   </joint>
@@ -163,10 +150,3 @@
     <parent link="rg6_g_main"/><child link="rg6_hand_tcp"/>
   </joint>
-  <!--
-    AUF/ZU-ANIMATION: aktiv. Treiber 'rg6-l_out_joint' wird vom
-    rg6_joint_state_broadcaster aus tool_data.analog_input2 gespeist. Damit der
-    Greifer animiert, muss dessen joint_states auf dem Topic landen, das der
-    Greifer-rendernde robot_state_publisher konsumiert (siehe rg6_bringup.launch.py
-    Argument 'js_topic').
-  -->
 </robot>

Commit message: Change RG6 model

File: src/rg6_description/urdf/clearpath_extras.urdf.xacro (robot description, xacro)
@@ -10,23 +10,17 @@
     - arm_0_tool0   = UR5 Tool-Frame (ROS-Industrial all-zeros)  -> RG6-Greifer
     - default_mount = Frame, auf dem der ArUco-Marker sitzt (TODO anpassen)
-  WICHTIG:
-    * Alle Greifer-Links sind mit 'rg6_' praefixiert -> KEINE Kollision mit base_link.
-    * rg6_description muss in einem in robot.yaml eingetragenen Workspace liegen.
-  ANIMATION (Auf/Zu):
-    Die RG6-Meshes sind im SolidWorks-Export ALLE im Basis-Frame authored (jedes
-    Mesh sitzt korrekt, wenn es bei xyz=0 an rg6_base_link haengt). Die reale
-    Kinematik ist ein 4-Gelenk-Parallelogramm pro Finger; das laesst sich im
-    URDF-Baum nur ungenau per mimic abbilden und ZERFAELLT bei Bewegung.
-    Daher hier vereinfacht: jeder Finger = EIN starrer Link (out+tip+inner), der um
-    sein Aussengelenk schwenkt. Treibergelenk 'rg6-l_out_joint' wird vom
-    rg6_joint_state_broadcaster aus tool_data.analog_input2 gespeist; der rechte
-    Finger folgt per <mimic multiplier="-1"> -> symmetrisches Auf/Zu, nichts zerfaellt.
-    Pivot/Visual-Offsets sind die globalen Aussengelenk-Positionen:
-        links  = base->g_main + g_main->l_out = (0.023851, 0.012801, 0.13453)
-        rechts = base->g_main + g_main->r_out = (-0.023749, 0.012801, 0.13453)
+  GREIFERMODELL:
+    Sauber artikuliertes RG6 aus package 'onrobot_rg6_visualization' (Robotiq-Stil:
+    outer_knuckle/inner_knuckle/inner_finger pro Seite, getrennte visual/collision-
+    Meshes). Treibergelenk = 'rg6_finger_joint' (Praefix 'rg6_'): 0 = offen,
+    positiv = zu. Alle anderen Greifergelenke folgen per <mimic> -> die
+    Parallelogramm-Schleife bleibt geschlossen, nichts zerfaellt.
+    Der rg6_joint_state_broadcaster speist 'rg6_finger_joint'.
+  VORAUSSETZUNG: sowohl 'rg6_description' (falls weiter genutzt) als auch
+  'onrobot_rg6_visualization' muessen in einem in robot.yaml unter
+  'system.ros2.workspaces' eingetragenen Workspace installiert sein, sonst findet
+  die foxglove_bridge die package://-Meshes nicht.
 -->
 <robot xmlns:xacro="http://ros.org/wiki/xacro">
-  <xacro:include filename="$(find rg6_description)/urdf/materials.xacro"/>
-  <material name="black"><color rgba="0.165 0.165 0.165 1.0"/></material>
   <material name="white"><color rgba="0.9137 0.9137 0.9137 1.0"/></material>
   <!-- =========================== ArUco-Marker =========================== -->
@@ -44,109 +38,21 @@
   </joint>
   <!-- ===================== RG6-Greifer an arm_0_tool0 =================== -->
-  <!-- rpy: Roll -90deg um X (empirisch bestaetigt fuer arm_0_tool0). -->
+  <!-- Greifermodell instanziieren (Praefix 'rg6_'). -->
+  <xacro:include filename="$(find onrobot_rg6_visualization)/urdf/onrobot_rg6_model_macro.xacro"/>
+  <xacro:onrobot_rg6 prefix="rg6_"/>
+  <!-- Greiferbasis an den Tool-Flansch.
+       rpy ggf. anpassen (in Foxglove pruefen): das neue Modell hat ein anderes
+       Mesh-Frame als das alte; Startwert 0 0 0. Falls verkippt/verdreht, je 90deg:
+         rpy="-1.5708 0 0" | rpy="1.5708 0 0" | rpy="0 0 1.5708" ... -->
   <joint name="rg6_tool0_to_base" type="fixed">
     <parent link="arm_0_tool0"/>
-    <child link="rg6_base_link"/>
-    <origin xyz="0 0 0" rpy="-1.5708 0 0"/>
+    <child link="rg6_onrobot_rg6_base_link"/>
+    <origin xyz="0 0 0" rpy="0 0 0"/>
   </joint>
-  <!-- ===== statische Teile ===== -->
-  <link name="rg6_base_link">
-    <visual>
-      <origin xyz="0 0 0" rpy="0 0 0"/>
-      <geometry><mesh filename="package://rg6_description/meshes/base_link.stl" scale="0.001 0.001 0.001"/></geometry>
-      <material name="silver"/>
-    </visual>
-    <collision>
-      <origin xyz="0 0 0" rpy="0 0 0"/>
-      <geometry><mesh filename="package://rg6_description/meshes/base_link.stl" scale="0.001 0.001 0.001"/></geometry>
-    </collision>
-  </link>
-  <link name="rg6_g_main">
-    <visual>
-      <origin xyz="0.031849 -1e-06 -0.04953" rpy="0 0 0"/>
-      <geometry><mesh filename="package://rg6_description/meshes/g_main.stl" scale="0.001 0.001 0.001"/></geometry>
-      <material name="silver"/>
-    </visual>
-    <collision>
-      <origin xyz="0.031849 -1e-06 -0.04953" rpy="0 0 0"/>
-      <geometry><mesh filename="package://rg6_description/meshes/g_main.stl" scale="0.001 0.001 0.001"/></geometry>
-    </collision>
-  </link>
-  <!-- ===== linker Finger als EIN starrer Link (out + tip + inner) ===== -->
-  <link name="rg6_left_finger">
-    <visual>
-      <origin xyz="-0.023851 -0.012801 -0.13453" rpy="0 0 0"/>
-      <geometry><mesh filename="package://rg6_description/meshes/l_out.stl" scale="0.001 0.001 0.001"/></geometry>
-      <material name="silver"/>
-    </visual>
-    <visual>
-      <origin xyz="-0.023851 -0.012801 -0.13453" rpy="0 0 0"/>
-      <geometry><mesh filename="package://rg6_description/meshes/l_inner.stl" scale="0.001 0.001 0.001"/></geometry>
-      <material name="silver"/>
-    </visual>
-    <visual>
-      <origin xyz="-0.023851 -0.012801 -0.13453" rpy="0 0 0"/>
-      <geometry><mesh filename="package://rg6_description/meshes/l_tip.stl" scale="0.001 0.001 0.001"/></geometry>
-      <material name="black"/>
-    </visual>
-    <collision>
-      <origin xyz="-0.023851 -0.012801 -0.13453" rpy="0 0 0"/>
-      <geometry><mesh filename="package://rg6_description/meshes/l_out.stl" scale="0.001 0.001 0.001"/></geometry>
-    </collision>
-    <collision>
-      <origin xyz="-0.023851 -0.012801 -0.13453" rpy="0 0 0"/>
-      <geometry><mesh filename="package://rg6_description/meshes/l_tip.stl" scale="0.001 0.001 0.001"/></geometry>
-    </collision>
-  </link>
-  <!-- ===== rechter Finger als EIN starrer Link (out + tip + inner) ===== -->
-  <link name="rg6_right_finger">
-    <visual>
-      <origin xyz="0.023749 -0.012801 -0.13453" rpy="0 0 0"/>
-      <geometry><mesh filename="package://rg6_description/meshes/r_out.stl" scale="0.001 0.001 0.001"/></geometry>
-      <material name="silver"/>
-    </visual>
-    <visual>
-      <origin xyz="0.023749 -0.012801 -0.13453" rpy="0 0 0"/>
-      <geometry><mesh filename="package://rg6_description/meshes/r_inner.stl" scale="0.001 0.001 0.001"/></geometry>
-      <material name="silver"/>
-    </visual>
-    <visual>
-      <origin xyz="0.023749 -0.012801 -0.13453" rpy="0 0 0"/>
-      <geometry><mesh filename="package://rg6_description/meshes/r_tip.stl" scale="0.001 0.001 0.001"/></geometry>
-      <material name="black"/>
-    </visual>
-    <collision>
-      <origin xyz="0.023749 -0.012801 -0.13453" rpy="0 0 0"/>
-      <geometry><mesh filename="package://rg6_description/meshes/r_out.stl" scale="0.001 0.001 0.001"/></geometry>
-    </collision>
-    <collision>
-      <origin xyz="0.023749 -0.012801 -0.13453" rpy="0 0 0"/>
-      <geometry><mesh filename="package://rg6_description/meshes/r_tip.stl" scale="0.001 0.001 0.001"/></geometry>
-    </collision>
-  </link>
-  <!-- ===== Gelenke ===== -->
-  <joint name="rg6_g_main_joint" type="fixed">
-    <origin xyz="-0.031849 1e-06 0.04953" rpy="0 0 0"/>
-    <parent link="rg6_base_link"/><child link="rg6_g_main"/>
-  </joint>
-  <!-- TREIBER: vom rg6_joint_state_broadcaster gesetzt. Pivot = linkes Aussengelenk. -->
-  <joint name="rg6-l_out_joint" type="revolute">
-    <origin xyz="0.023851 0.012801 0.13453" rpy="0 0 0"/>
-    <parent link="rg6_base_link"/><child link="rg6_left_finger"/>
-    <axis xyz="0 1 0"/>
-    <limit upper="0.610865" lower="-0.75" effort="100" velocity="100"/>
-  </joint>
-  <joint name="rg6_right_finger_joint" type="revolute">
-    <origin xyz="-0.023749 0.012801 0.13453" rpy="0 0 0"/>
-    <parent link="rg6_base_link"/><child link="rg6_right_finger"/>
-    <axis xyz="0 1 0"/>
-    <limit upper="0.610865" lower="-0.75" effort="100" velocity="100"/>
-    <mimic joint="rg6-l_out_joint" multiplier="-1"/>
-  </joint>
-  <!-- Greifer-TCP -->
+  <!-- Greifer-TCP (mittig zwischen den Fingerspitzen, grob). -->
   <link name="rg6_hand_tcp"/>
   <joint name="rg6_hand_tcp_joint" type="fixed">
-    <origin xyz="0.036 0 0.21" rpy="0 0 0"/>
-    <parent link="rg6_g_main"/><child link="rg6_hand_tcp"/>
+    <origin xyz="0 0 0.21" rpy="0 0 0"/>
+    <parent link="rg6_onrobot_rg6_base_link"/><child link="rg6_hand_tcp"/>
   </joint>
 </robot>
