Commit message: Fix RG6 broadcaster

File: src/rg6_description/urdf/clearpath_extras.urdf.xacro (robot description, xacro)
@@ -41,12 +41,11 @@
   <xacro:include filename="$(find onrobot_rg6_visualization)/urdf/onrobot_rg6_model_macro.xacro"/>
   <xacro:onrobot_rg6 prefix="rg6_"/>
-  <!-- Greiferbasis an den Tool-Flansch.
-       rpy ggf. anpassen (in Foxglove pruefen): das neue Modell hat ein anderes
-       Mesh-Frame als das alte; Startwert 0 0 0. Falls verkippt/verdreht, je 90deg:
-         rpy="-1.5708 0 0" | rpy="1.5708 0 0" | rpy="0 0 1.5708" ... -->
+  <!-- Greiferbasis an den Tool-Flansch. Modell-Achse = +Z (wie altes Modell),
+       daher Roll -90deg um X. Falls noch verdreht, je 90deg variieren:
+         rpy="1.5708 0 0" | rpy="0 0 1.5708" | rpy="0 0 -1.5708" -->
   <joint name="rg6_tool0_to_base" type="fixed">
     <parent link="arm_0_tool0"/>
     <child link="rg6_onrobot_rg6_base_link"/>
-    <origin xyz="0 0 0" rpy="0 0 0"/>
+    <origin xyz="0 0 0" rpy="-1.5708 0 0"/>
   </joint>
   <!-- Greifer-TCP (mittig zwischen den Fingerspitzen, grob). -->

Commit message: Test rotation change

File: src/rg6_description/urdf/clearpath_extras.urdf.xacro (robot description, xacro)
@@ -47,5 +47,5 @@
     <parent link="arm_0_tool0"/>
     <child link="rg6_onrobot_rg6_base_link"/>
-    <origin xyz="0 0 0" rpy="0 0 0"/>
+    <origin xyz="0 0 0" rpy="0 1.5708 0"/>
   </joint>
   <!-- Greifer-TCP (mittig zwischen den Fingerspitzen, grob). -->

Commit message: Test rotation change

File: src/rg6_description/urdf/clearpath_extras.urdf.xacro (robot description, xacro)
@@ -47,5 +47,5 @@
     <parent link="arm_0_tool0"/>
     <child link="rg6_onrobot_rg6_base_link"/>
-    <origin xyz="0 0 0" rpy="0 1.5708 0"/>
+    <origin xyz="0 0 0" rpy="0 0 1.5708"/>
   </joint>
   <!-- Greifer-TCP (mittig zwischen den Fingerspitzen, grob). -->

Commit message: Set final rotation to RG6

File: src/rg6_description/urdf/clearpath_extras.urdf.xacro (robot description, xacro)
@@ -47,5 +47,5 @@
     <parent link="arm_0_tool0"/>
     <child link="rg6_onrobot_rg6_base_link"/>
-    <origin xyz="0 0 0" rpy="0 0 1.5708"/>
+    <origin xyz="0 0 0" rpy="0 0 -1.5708"/>
   </joint>
   <!-- Greifer-TCP (mittig zwischen den Fingerspitzen, grob). -->

Commit message: Add sensor arch

File: src/rg6_description/urdf/clearpath_extras.urdf.xacro (robot description, xacro)
@@ -55,3 +55,18 @@
     <parent link="rg6_onrobot_rg6_base_link"/><child link="rg6_hand_tcp"/>
   </joint>
+  <!-- ===== Custom Top-Assembly (ersetzt a200.sensor_arch) ===== -->
+  <link name="husky_top_assembly">
+    <visual>
+      <origin xyz="0 0 0" rpy="0 0 0"/>
+      <geometry>
+        <mesh filename="package://onrobot_rg6_visualization/meshes/husky_top_assembly.dae"/>
+        <!-- falls nicht in Metern exportiert: scale="0.001 0.001 0.001" am mesh ergaenzen -->
+      </geometry>
+    </visual>
+  </link>
+  <joint name="husky_top_assembly_joint" type="fixed">
+    <parent link="default_mount"/>      <!-- TODO: realer Mount-Frame aus Schritt 1 -->
+    <child link="husky_top_assembly"/>
+    <origin xyz="0 0 0" rpy="0 0 0"/>   <!-- TODO: Offset aus Schritt 1 -->
+  </joint>
 </robot>

Commit message: Change sensor arch model

File: src/rg6_description/urdf/clearpath_extras.urdf.xacro (robot description, xacro)
@@ -60,5 +60,5 @@
       <origin xyz="0 0 0" rpy="0 0 0"/>
       <geometry>
-        <mesh filename="package://onrobot_rg6_visualization/meshes/husky_top_assembly.dae"/>
+        <mesh filename="package://onrobot_rg6_visualization/meshes/husky_sensor_arch.stl"/>
         <!-- falls nicht in Metern exportiert: scale="0.001 0.001 0.001" am mesh ergaenzen -->
       </geometry>

Commit message: Fix positions in urdf

File: src/rg6_description/urdf/clearpath_extras.urdf.xacro (robot description, xacro)
@@ -28,12 +28,12 @@
   <link name="aruco_marker">
     <visual>
-      <geometry><box size="0.127 0.127 0.001"/></geometry>
+      <geometry><box size="0.11 0.11 0.001"/></geometry>
       <material name="white"/>
     </visual>
   </link>
   <joint name="aruco_to_base" type="fixed">
-    <parent link="default_mount"/>          <!-- TODO: korrektes Frame -->
+    <parent link="top_plate_front_mount"/>          <!-- TODO: korrektes Frame -->
     <child link="aruco_marker"/>
-    <origin rpy="0 0 0" xyz="0.048 -0.134 0"/>  <!-- TODO: realer Offset -->
+    <origin rpy="0 0 0" xyz="-0.062 -0.142 0"/>  <!-- TODO: realer Offset -->
   </joint>
   <!-- ===================== RG6-Greifer an arm_0_tool0 =================== -->
@@ -58,19 +58,15 @@
   <link name="husky_top_assembly">
     <visual>
-      <!-- Visual-Origin "nullt" das Mesh: rpy dreht es aufrecht, xyz schiebt den
-           Fuss-Mittelpunkt auf den Link-Ursprung (CAD-Versatz nach Drehung:
-           x 0.31, y 0.30, z -0.265 -> Gegenvektor hier). -->
-      <origin xyz="-0.31 -0.30 0.265" rpy="-1.5708 0 0"/>
+      <origin xyz="0 0 0" rpy="0 0 -1.5708"/>
       <geometry>
         <mesh filename="package://onrobot_rg6_visualization/meshes/husky_sensor_arch.stl"/>
+        <!-- falls nicht in Metern exportiert: scale="0.001 0.001 0.001" am mesh ergaenzen -->
       </geometry>
     </visual>
   </link>
   <joint name="husky_top_assembly_joint" type="fixed">
-    <parent link="top_plate_back_mount"/>
+    <parent link="top_plate_rear_mount"/>
     <child link="husky_top_assembly"/>
-    <!-- Origin 0 0 0 = Fuss-Mittelpunkt sitzt exakt auf top_plate_back_mount.
-         Hier intuitiv nachschieben (z hoch, x vor/zurueck, y links/rechts). -->
-    <origin xyz="0 0 0" rpy="0 0 0"/>
+    <origin xyz="0 0.315 0" rpy="0 0 0"/>
   </joint>
 </robot>

Commit message: Change STL to GLTF model

File: src/rg6_description/urdf/clearpath_extras.urdf.xacro (robot description, xacro)
@@ -57,9 +57,12 @@
   <!-- ===== Custom Top-Assembly (ersetzt a200.sensor_arch) ===== -->
   <link name="husky_top_assembly">
+    <!-- glTF (selbst-enthaltend, 2 Materialien) statt STL -> Materialien sichtbar.
+         KEIN <material> hier setzen, sonst werden die glTF-Materialien ueberschrieben.
+         Hinweis: glTF ist Y-up (Onshape-Export); falls das Modell ggue. der STL um
+         90deg verkippt erscheint, rpy nachziehen (typisch +/-1.5708 um X). -->
     <visual>
       <origin xyz="0 0 0" rpy="0 0 -1.5708"/>
       <geometry>
-        <mesh filename="package://onrobot_rg6_visualization/meshes/husky_sensor_arch.stl"/>
-        <!-- falls nicht in Metern exportiert: scale="0.001 0.001 0.001" am mesh ergaenzen -->
+        <mesh filename="package://onrobot_rg6_visualization/meshes/husky_sensor_arch.gltf"/>
       </geometry>
     </visual>

Commit message: Clean up and refactor

File: src/rg6_description/urdf/clearpath_extras.urdf.xacro (robot description, xacro)
@@ -11,12 +11,11 @@
     - default_mount = Frame, auf dem der ArUco-Marker sitzt (TODO anpassen)
   GREIFERMODELL:
-    Sauber artikuliertes RG6 aus package 'onrobot_rg6_visualization' (Robotiq-Stil:
-    outer_knuckle/inner_knuckle/inner_finger pro Seite, getrennte visual/collision-
-    Meshes). Treibergelenk = 'rg6_finger_joint' (Praefix 'rg6_'): 0 = offen,
-    positiv = zu. Alle anderen Greifergelenke folgen per <mimic> -> die
-    Parallelogramm-Schleife bleibt geschlossen, nichts zerfaellt.
-    Der rg6_joint_state_broadcaster speist 'rg6_finger_joint'.
-  VORAUSSETZUNG: sowohl 'rg6_description' (falls weiter genutzt) als auch
-  'onrobot_rg6_visualization' muessen in einem in robot.yaml unter
+    Sauber artikuliertes RG6 aus package 'rg6_description' (Robotiq-Stil:
+    outer_knuckle/inner_knuckle/inner_finger pro Seite). Treibergelenk =
+    'rg6_finger_joint' (Praefix 'rg6_'): 0 = offen, positiv = zu. Der
+    rg6_joint_state_broadcaster setzt ALLE 6 Greifergelenke EXPLIZIT (kein
+    <mimic> - das loesen manche URDF-Parser/Foxglove nicht zuverlaessig auf).
+    Kollision = eine grobe Box am base_link (keine Selbstkollision in MoveIt).
+  VORAUSSETZUNG: 'rg6_description' muss in einem in robot.yaml unter
   'system.ros2.workspaces' eingetragenen Workspace installiert sein, sonst findet
   die foxglove_bridge die package://-Meshes nicht.
@@ -39,5 +38,5 @@
   <!-- ===================== RG6-Greifer an arm_0_tool0 =================== -->
   <!-- Greifermodell instanziieren (Praefix 'rg6_'). -->
-  <xacro:include filename="$(find onrobot_rg6_visualization)/urdf/onrobot_rg6_model_macro.xacro"/>
+  <xacro:include filename="$(find rg6_description)/urdf/onrobot_rg6_model_macro.xacro"/>
   <xacro:onrobot_rg6 prefix="rg6_"/>
   <!-- Greiferbasis an den Tool-Flansch. Modell-Achse = +Z (wie altes Modell),
@@ -64,5 +63,5 @@
       <origin xyz="0 0 0" rpy="0 0 -1.5708"/>
       <geometry>
-        <mesh filename="package://onrobot_rg6_visualization/meshes/husky_sensor_arch.gltf"/>
+        <mesh filename="package://rg6_description/meshes/husky_sensor_arch.gltf"/>
       </geometry>
     </visual>

File: src/rg6_description/urdf/onrobot_rg6.xacro (robot description, xacro)
@@ -11,5 +11,5 @@
         <origin xyz="0 0 0" rpy="0 0 0" />
         <geometry>
-          <mesh filename="package://onrobot_rg6_visualization/meshes/visual/base_link.stl" />
+          <mesh filename="package://rg6_description/meshes/visual/base_link.stl" />
         </geometry>
         <material name="rg6_silver">

File: src/rg6_description/urdf/onrobot_rg6_model.xacro (robot description, xacro)
@@ -1,5 +1,5 @@
 <?xml version="1.0"?>
 <robot name="onrobot_rg6_model" xmlns:xacro="http://ros.org/wiki/xacro">
-  <xacro:include filename="$(find onrobot_rg6_visualization)/urdf/onrobot_rg6_model_macro.xacro" />
+  <xacro:include filename="$(find rg6_description)/urdf/onrobot_rg6_model_macro.xacro" />
   <xacro:onrobot_rg6 prefix=""/>
 </robot>

File: src/rg6_description/urdf/onrobot_rg6_model_macro.xacro (robot description, xacro)
@@ -14,5 +14,5 @@
         <origin xyz="0 0 0" rpy="0 0 0" />
         <geometry>
-          <mesh filename="package://onrobot_rg6_visualization/meshes/visual/outer_knuckle.stl" />
+          <mesh filename="package://rg6_description/meshes/visual/outer_knuckle.stl" />
         </geometry>
         <material name="rg6_silver">
@@ -34,5 +34,5 @@
         <origin xyz="0 0 0" rpy="0 0 0" />
         <geometry>
-          <mesh filename="package://onrobot_rg6_visualization/meshes/visual/inner_knuckle.stl" />
+          <mesh filename="package://rg6_description/meshes/visual/inner_knuckle.stl" />
         </geometry>
         <material name="rg6_silver">
@@ -53,5 +53,5 @@
         <origin xyz="0 0 0" rpy="0 0 0" />
         <geometry>
-          <mesh filename="package://onrobot_rg6_visualization/meshes/visual/inner_finger.stl" />
+          <mesh filename="package://rg6_description/meshes/visual/inner_finger.stl" />
         </geometry>
         <material name="rg6_black">
@@ -80,5 +80,5 @@
     </joint>
   </xacro:macro>
-  <xacro:include filename="$(find onrobot_rg6_visualization)/urdf/onrobot_rg6.xacro" />
+  <xacro:include filename="$(find rg6_description)/urdf/onrobot_rg6.xacro" />
   <xacro:macro name="finger_joint" params="prefix">
     <joint name="${prefix}finger_joint" type="revolute">
